File: defcon_badge_main/defcon_badge_main.kicad_pcb (KiCad board)
At the start: 2 copper layers, 63 x 41 mm, 146 parts, among them J1 USB_C_Receptacle, J10 Conn_01x02_Pin, J11 Conn_01x02_Pin, J12 Conn_01x02_Pin, J13 Conn_01x02_Pin, J14 Conn_01x02_Pin, J15 Conn_01x02_Pin, J16 Conn_01x02_Pin, J17 Conn_01x02_Pin, J18 Conn_01x02_Pin, J19 Conn_01x02_Pin, J20 Conn_01x02_Pin, J21 Conn_01x02_Pin, J22 Conn_01x02_Pin, J3 Conn_01x02_Pin, J9 Conn_01x02_Pin, M1 Motor 1, M2 Motor 2, M3 Motor 3, U3 ESP32-C5-WROOM-1U, U5 DRIVER-A4988SETTR-T_QFN28_, U6 DRIVER-A4988SETTR-T_QFN28_, U8 DRIVER-A4988SETTR-T_QFN28_

Commit message: begin full layout
Parts:
- added D1: PESD0402, PCM_SparkFun-Capacitor:C_0402_1005Metric, F.Cu at (198.0, 40.0)
- added D2: PESD0402, PCM_SparkFun-Capacitor:C_0402_1005Metric, F.Cu at (199.5, 42.5)
- added J4: Conn_01x02_Pin, Connector_PinHeader_1.00mm:PinHeader_1x02_P1.00mm_Vertical, F.Cu at (274.6, 167.8)
- added J5: Conn_01x02_Pin, Connector_PinHeader_1.00mm:PinHeader_1x02_P1.00mm_Vertical, F.Cu at (277.9, 167.8)
- added J6: Conn_01x02_Pin, Connector_PinHeader_1.00mm:PinHeader_1x02_P1.00mm_Vertical, F.Cu at (281.2, 167.8)
- R1_CS_M1, R1_CS_M2, R1_CS_M3, R2_CS_M1, R2_CS_M2, R2_CS_M3, R_BOOT1, R_EN_M1, R_EN_M2, R_EN_M3, R_M1, R_M2, R_M3, R_RST_M1, R_RST_M2, R_RST_M3, R_SLP_M1, R_SLP_M2, R_SLP_M3, R_SNS1_M1, R_SNS1_M2, R_SNS1_M3, R_SNS2_M1, R_SNS2_M2, R_SNS2_M3: footprint PCM_SparkFun-Fuse:1206 -> PCM_SparkFun-Coil:0805
- R_USB_D+1, R_USB_D-1, R_USB_PUPD+1, R_USB_PUPD-1: footprint PCM_SparkFun-Coil:0805 -> Resistor_SMD:R_0402_1005Metric
- SW_BOOT1, SW_EN1: footprint Button_Switch_SMD:SW_SPST_PTS645 -> Button_Switch_SMD:SW_SPST_PTS810
- moved J1 181.4 mm to (200.3, 40.2), turned to 120 degrees
- moved R_USB_CC2 181.3 mm to (198.0, 34.0), turned to -150 degrees
- moved R_USB_CC1 174.9 mm to (204.5, 45.5), turned to 30 degrees
- moved R_USB_PUPD+1 165.2 mm to (192.5, 40.5), turned to 90 degrees
- moved C_USB_D+1 162.5 mm to (191.0, 40.5), turned to 90 degrees
- moved R_USB_PUPD-1 160.5 mm to (192.5, 43.0), turned to -90 degrees
- moved C_USB_D-1 158.3 mm to (191.0, 43.0), turned to -90 degrees
- moved R_USB_D+1 158.3 mm to (189.0, 41.0)
- moved SW_EN1 156.3 mm to (181.0, 33.5), turned to 180 degrees
- moved R1_EN1 155.9 mm to (188.5, 32.5)
- moved R_USB_D-1 155.2 mm to (189.0, 42.5), turned to 0 degrees
- moved C1_EN1 154.7 mm to (185.5, 33.5), turned to -90 degrees
- moved C2_EN1 143.9 mm to (192.0, 53.5)
- moved R2_EN1 141.3 mm to (193.5, 55.5), turned to -90 degrees
- moved C2_DC3 137.9 mm to (189.5, 57.6), turned to -90 degrees
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Routing:
- net /3v3: track 33.5 -> 0.00 mm
- net /esp32/boot2: track 32.9 -> 0.00 mm
- net GND: track 20.2 -> 0.00 mm, vias 38 -> 0
- net /STEPPER_3_DIR: track 19.9 -> 0.00 mm
- net /STEPPER_3_STEP: track 19.6 -> 0.00 mm
- net /MENU_SEL: track 19.0 -> 0.00 mm
- net /esp32/USB_D+: track 17.2 -> 0.00 mm
- net /esp32/USB_D-: track 17.0 -> 0.00 mm
- net /LIMIT_SWITCH: track 16.2 -> 0.00 mm
- net /esp32/I2C_SDA: track 14.6 -> 0.00 mm
- net Net-(U3-EN/CHIP_PU): track 12.5 -> 0.00 mm
- net /esp32/ESP_D-: track 11.0 -> 0.00 mm
- net /esp32/ESP_D+: track 10.8 -> 0.00 mm
- net /esp32/I2C_SCL: track 10.2 -> 0.00 mm
- net /STEPPER_2_STEP: track 9.02 -> 0.00 mm
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- removed copper zone on F.Cu, net /3v3
- removed copper zone on B.Cu, net GND
- removed copper zone on F.Cu, net GND
Other:
- board size 63 x 41 mm -> 102.5 x 89.5 mm
- copper layers 2 -> 4

Commit message: more layout
Parts:
- removed C_LIM2, C_LIM3, C_LIM4, C_LIM5, C_LIM6: 0.1 uF, PCM_SparkFun-Coil:0805
- removed D_LIM2, D_LIM3, D_LIM4, D_LIM5, D_LIM6: ~, PCM_SparkFun-Semiconductor-Standard:SOD-123
- removed R1_LIM2, R1_LIM3, R1_LIM4, R1_LIM5, R1_LIM6: 10 kOhm, PCM_SparkFun-Fuse:1206
- removed R2_LIM2, R2_LIM3, R2_LIM4, R2_LIM5, R2_LIM6: 1 kOhm, PCM_SparkFun-Fuse:1206
- BT1: moved to B.Cu
- C1_CHR_M1, C1_CHR_M2, C1_CHR_M3, C1_M1, C1_M2, C1_M3, C2_M1, C2_M2, C2_M3, C3_M1, C3_M2, C3_M3, R1_CS_M1, R1_CS_M2, R1_CS_M3, R2_CS_M1, R2_CS_M2, R2_CS_M3, R_EN_M1, R_EN_M2, R_EN_M3, R_M1, R_M2, R_M3, R_RST_M1, R_RST_M2, R_RST_M3, R_SNS1_M1, R_SNS1_M2, R_SNS1_M3, R_SNS2_M1, R_SNS2_M2, R_SNS2_M3: footprint PCM_SparkFun-Coil:0805 -> joystick:R_0603_1608Metric_Pad0.98x0.95mm_HandSolder_MINE
- C1_DC3, C1_EN1, C1_V3, C1_V5, C1_V8, C2_DC3, C2_EN1, C2_V3, C2_V5, C3_V8, C_BOOT1, C_LIM1, C_MENU1, R1_EN1, R2_EN1, R_BOOT1, R_MENU1, R_USB_CC1, R_USB_CC2: footprint PCM_SparkFun-Coil:0805 -> joystick:R_0805_2012Metric_Pad1.20x1.40mm_HandSolder_MINE
- C2_V8, C_USB_D+1, C_USB_D-1: footprint Capacitor_SMD:C_0402_1005Metric -> joystick:R_0402_1005Metric_Pad0.72x0.64mm_HandSolder_MINE
- D1, D2: footprint PCM_SparkFun-Capacitor:C_0402_1005Metric -> joystick:R_0402_1005Metric_Pad0.72x0.64mm_HandSolder_MINE
- R1_BLED1, R1_GLED1, R1_LIM1, R1_RLED1, R1_V3, R1_V5, R1_V8, R2_BLED1, R2_GLED1, R2_LIM1, R2_RLED1, R2_V3, R2_V5, R2_V8, R3_V8: footprint PCM_SparkFun-Fuse:1206 -> joystick:R_1206_3216Metric_Pad1.30x1.75mm_HandSolder_MINE
- R_OSC_M1: renamed from R_SLP_M1; footprint PCM_SparkFun-Coil:0805 -> joystick:R_0603_1608Metric_Pad0.98x0.95mm_HandSolder_MINE
- R_OSC_M2: renamed from R_SLP_M2; footprint PCM_SparkFun-Coil:0805 -> joystick:R_0603_1608Metric_Pad0.98x0.95mm_HandSolder_MINE
- R_OSC_M3: renamed from R_SLP_M3; footprint PCM_SparkFun-Coil:0805 -> joystick:R_0603_1608Metric_Pad0.98x0.95mm_HandSolder_MINE
- R_USB_D+1, R_USB_D-1, R_USB_PUPD+1, R_USB_PUPD-1: footprint Resistor_SMD:R_0402_1005Metric -> joystick:R_0402_1005Metric_Pad0.72x0.64mm_HandSolder_MINE
- moved Q_BLED1 209.6 mm to (130.6, 24.7)
- moved R1_BLED1 193.1 mm to (135.5, 23.2), turned to 180 degrees
- moved RED_1 155.7 mm to (129.8, 110.6), turned to 180 degrees
- moved R1_GLED1 149.6 mm to (156.8, 65.4)
- moved R2_LIM1 148.6 mm to (195.6, 63.6), turned to -90 degrees
- moved GREEN_1 148.4 mm to (135.2, 127.0)
- moved D_LIM1 148.1 mm to (193.2, 65.5), turned to -90 degrees
- moved R1_LIM1 143.0 mm to (195.6, 58.3), turned to -90 degrees
- moved C_LIM1 142.1 mm to (193.2, 59.4), turned to -90 degrees
- moved R_MENU1 137.4 mm to (152.3, 41.5), turned to 90 degrees
- moved C_MENU1 135.3 mm to (154.8, 41.5), turned to -90 degrees
- moved R_SNS2_M1 127.9 mm to (154.7, 90.9), turned to 90 degrees
- moved J_LIM1 124.9 mm to (185.2, 62.9), turned to 30 degrees
- moved C1_M1 124.8 mm to (151.1, 97.9), turned to 90 degrees
- moved L_V8 124.1 mm to (216.7, 77.5), turned to -90 degrees
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- renumbered J6 to BLUE_1, J18 to BLUE_2, J19 to BLUE_3, J20 to BLUE_4, J21 to BLUE_5, J22 to BLUE_6, J5 to GREEN_1, J13 to GREEN_2, J14 to GREEN_3, J15 to GREEN_4, J16 to GREEN_5, J17 to GREEN_6, J4 to RED_1, J3 to RED_2, J9 to RED_3, J10 to RED_4, J11 to RED_5, J12 to RED_6
Connections:
- net /3v3_power/VBAT renamed /VBAT
- net /esp32/ESP_D+ renamed /esp32/ESP_D_P
- net /esp32/ESP_D- renamed /esp32/ESP_D_N
- net /esp32/USB_D+ renamed /esp32/USB_D_P
- net /esp32/USB_D- renamed /esp32/USB_D_N
- net Net-(C1_EN1-Pad1) renamed /esp32/SW_EN
- net Net-(R_BOOT1-Pad1) renamed /esp32/boot2_sw
- net Net-(U3-EN/CHIP_PU) renamed /esp32/EN
- net Net-(U_3V1-FB) renamed /3v3_power/3v3_FB
- net Net-(U_3V1-SW) renamed /3v3_power/3v3_SW
- net Net-(U_5V1-FB) renamed /5v_power/5v_FB
- net Net-(U_5V1-SW) renamed /5v_power/5v_SW
- net Net-(U_V8-EN) renamed /8v_power/8v_EN
- net Net-(U_V8-FB) renamed /8v_power/8v_FB
- net Net-(U_V8-SW) renamed /8v_power/8v_SW
- J_LIM1 pad 2: Net-(J_LIM1-Pin_2) -> /limit_switch/SW_PARALLEL
- J_LIM2 pad 2: Net-(J_LIM2-Pin_2) -> /limit_switch/SW_PARALLEL
- J_LIM3 pad 2: Net-(J_LIM3-Pin_2) -> /limit_switch/SW_PARALLEL
- J_LIM4 pad 2: Net-(J_LIM4-Pin_2) -> /limit_switch/SW_PARALLEL
- J_LIM5 pad 2: Net-(J_LIM5-Pin_2) -> /limit_switch/SW_PARALLEL
- J_LIM6 pad 2: Net-(J_LIM6-Pin_2) -> /limit_switch/SW_PARALLEL
- R2_LIM1 pad 2: Net-(J_LIM1-Pin_2) -> /limit_switch/SW_PARALLEL
- U3 pad 10: /LIMIT_SWITCH -> /STEPPER_2_STEP
- U3 pad 16: /JOY_Y -> /JOY_X
- U3 pad 17: /JOY_X -> /JOY_Y
- U3 pad 24: /STEPPER_1_STEP -> /STEPPER_1_DIR
- U3 pad 25: /STEPPER_1_DIR -> /STEPPER_1_STEP
- U3 pad 6: /STEPPER_2_STEP -> /LIMIT_SWITCH
- U3 pad 7: /STEPPER_2_DIR -> /STEPPER_3_DIR
- U3 pad 9: /STEPPER_3_DIR -> /STEPPER_2_DIR
- U_V8 pad 1: unconnected-(U_V8-PGND-Pad1) -> GND
- U_V8 pad 5: unconnected-(U_V8-AGND-Pad5) -> GND
- U_V8 pad 7: unconnected-(U_V8-PAD-Pad7) -> GND
Routing:
- net /STEPPER_MS2: track 0.00 -> 147.8 mm, vias 0 -> 8
- net /STEPPER_MS3: track 0.00 -> 147.2 mm, vias 0 -> 8
- net /STEPPER_MS1: track 0.00 -> 145.2 mm, vias 0 -> 8
- net /esp32/I2C_SDA: track 0.00 -> 101.5 mm, vias 0 -> 3
- net /esp32/I2C_SCL: track 0.00 -> 96.8 mm, vias 0 -> 3
- net /STEPPER_3_STEP: track 0.00 -> 77.8 mm, vias 0 -> 4
- net /STEPPER_2_STEP: track 0.00 -> 72.1 mm, vias 0 -> 2
- net /STEPPER_3_DIR: track 0.00 -> 70.4 mm, vias 0 -> 4
- net /STEPPER_2_DIR: track 0.00 -> 66.1 mm, vias 0 -> 2
- net /STEPPER_1_STEP: track 0.00 -> 61.7 mm, vias 0 -> 4
- net /STEPPER_1_DIR: track 0.00 -> 60.8 mm, vias 0 -> 4
- net /JOY_Y: track 0.00 -> 48.5 mm
- net /esp32/EN: track 0.00 -> 41.4 mm, vias 0 -> 2
- net /JOY_X: track 0.00 -> 38.5 mm
- net /MENU_SEL: track 0.00 -> 30.9 mm, vias 0 -> 2
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- added copper zone on In1.Cu, net (none)
- added copper zone on F.Cu, net /3v3
- added copper zone on In2.Cu, net /3v3
- added copper zone on F.Cu, net /3v3_power/3v3_FB
- added copper zone on F.Cu, net /3v3_power/3v3_SW
- added copper zone on F.Cu, net /5v
- added copper zone on F.Cu, net /5v_power/5v_FB
- added copper zone on F.Cu, net /5v_power/5v_SW
- added copper zone on F.Cu, net /8v
- added copper zone on In2.Cu, net /8v
- added copper zone on F.Cu, net /8v_power/8v_EN
- added copper zone on F.Cu, net /8v_power/8v_FB
- added copper zone on F.Cu, net /8v_power/8v_SW
- added copper zone on F.Cu, net /LIMIT_SWITCH
- added copper zone on F.Cu, net /MENU_SEL
- added copper zone on F.Cu, net /VBAT
- added copper zone on In2.Cu, net /VBAT
- added copper zone on F.Cu, net /esp32/SW_EN
- added copper zone on F.Cu, net /esp32/boot2
- added copper zone on F.Cu, net /esp32/boot2_sw
- added copper zone on F.Cu, net /limit_switch/SW_PARALLEL
- added copper zone on F.Cu, net /motor_driver/REF
- added copper zone on F.Cu, net /motor_driver1/REF
- added copper zone on F.Cu, net /motor_driver2/REF
- added copper zone on B.Cu, net GND
- added copper zone on F.Cu, net GND
- added copper zone on In1.Cu, net GND
- added copper zone on In2.Cu, net GND
Other:
- outline, holes or cut-outs redrawn

Commit message: moar layout
Parts:
- removed J1: USB_C_Receptacle, PCM_SparkFun-Connector:USB-C_16
- removed R_USB_CC1, R_USB_CC2: 5.1k Ohm, joystick:R_0805_2012Metric_Pad1.20x1.40mm_HandSolder_MINE
- added D_8V2: SS24FL, SS24FL:SODFL3617X108N, F.Cu at (31.3, -7.80)
- added REF**: limit_switch_mount, joystick:limit_switch_mount, F.Cu at (-15.1, -4.80)
- added U1: ~, joystick:usb_typea_boardedge, F.Cu at (49.0, -35.8)
- R1_BLED1, R1_GLED1, R1_RLED1, R2_BLED1, R2_GLED1, R2_RLED1: footprint joystick:R_1206_3216Metric_Pad1.30x1.75mm_HandSolder_MINE -> joystick:R_0805_2012Metric_Pad1.20x1.40mm_HandSolder
- moved BLUE_3 291.6 mm to (-22.9, -40.5), turned to -120 degrees
- moved GREEN_3 281.9 mm to (-25.3, -36.3), turned to -120 degrees
- moved BLUE_2 279.3 mm to (-46.5, -0.45), turned to -60 degrees
- moved GREEN_2 268.9 mm to (-44.1, 3.71), turned to -60 degrees
- moved Q_RLED1 268.3 mm to (-21.6, -37.1), turned to 180 degrees
- moved RED_2 267.1 mm to (-45.3, 1.63), turned to -60 degrees
- moved R2_RLED1 262.3 mm to (-20.0, -40.2), turned to -90 degrees
- moved GREEN_4 257.7 mm to (18.8, -39.9), turned to 180 degrees
- moved R2_GLED1 256.1 mm to (-24.7, -32.2)
- moved Q_GLED1 255.8 mm to (-22.2, -31.4), turned to -90 degrees
- moved RED_3 255.3 mm to (-24.1, -38.4), turned to -120 degrees
- moved R1_RLED1 247.2 mm to (-17.8, -34.7), turned to 180 degrees
- moved BLUE_1 244.7 mm to (-23.6, 40.1)
- moved BLUE_4 244.0 mm to (23.6, -39.9), turned to 180 degrees
- moved R2_BLED1 241.1 mm to (-13.4, -39.6), turned to 180 degrees
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Connections:
- net Net-(Q_BLED1-B) renamed /led/LED_B_SIG
- net Net-(Q_BLED1-C) renamed /led/LED_B_POW
- net Net-(Q_GLED1-B) renamed /led/LED_G_SIG
- net Net-(Q_GLED1-C) renamed /led/LED_G_POW
- net Net-(Q_RLED1-B) renamed /led/LED_R_SIG
- net Net-(Q_RLED1-C) renamed /led/LED_R_POW
- C2_V5 pad 1: /5v -> /5v_power/5v_out
- R1_V5 pad 1: /5v -> /5v_power/5v_out
- U_5V1 pad 6: /5v -> /5v_power/5v_out
Routing:
- net Net-(RED_1-Pin_1): track 0.00 -> 65.5 mm, vias 0 -> 2
- net Net-(BLUE_1-Pin_1): track 0.00 -> 62.8 mm, vias 0 -> 2
- net Net-(GREEN_1-Pin_1): track 0.00 -> 49.6 mm, vias 0 -> 1
- net /esp32/boot1: track 15.1 -> 4.32 mm, vias 2 -> 0
- net /STEPPER_MS1: track 145.2 -> 155.6 mm
- net /led/LED_G_SIG: track 0.00 -> 10.2 mm, vias 0 -> 2
- net /STEPPER_MS2: track 147.8 -> 157.4 mm
- net /STEPPER_MS3: track 147.2 -> 154.3 mm
- net /MENU_SEL: track 30.9 -> 35.0 mm
- net /led/LED_B_POW: track 0.00 -> 4.09 mm
- net /STEPPER_1_DIR: track 60.8 -> 64.3 mm
- net /STEPPER_1_STEP: track 61.7 -> 65.0 mm
- net /led/LED_R_SIG: track 0.00 -> 2.97 mm
- net /led/LED_R_POW: track 0.00 -> 2.85 mm
- net /esp32/boot2: track 0.00 -> 2.20 mm
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- added copper zone on In2.Cu, net /5v
- added copper zone on F.Cu, net /5v_power/5v_out
- removed copper zone on In1.Cu, net (none)
- removed copper zone on In2.Cu, net /VBAT
- removed copper zone on In1.Cu, net GND
Other:
- board size 102.5 x 89.5 mm -> 105.2 x 89.6 mm
- board text added: "0x1ea7bee5"

Commit message: done?
Parts:
- removed BT1: 1043P, 1043P:BAT_1043P
- added BT2: BK-18650-PC2, BK-18650-PC2:BAT_BK-18650-PC2, B.Cu at (-0.70, -0.10)
- moved U1 12.1 mm to (36.9, -35.1), turned to 30 degrees
- moved L_V8 0.55 mm to (39.5, 4.50)
- moved C1_V8 0.07 mm to (33.2, 1.09)
Routing:
- net Net-(GREEN_1-Pin_1): track 49.6 -> 292.2 mm, vias 1 -> 13
- net Net-(BLUE_1-Pin_1): track 62.8 -> 289.9 mm, vias 2 -> 8
- net Net-(RED_1-Pin_1): track 65.5 -> 285.1 mm, vias 2 -> 11
- net GND: track 1.84 -> 19.0 mm, vias 247 -> 368
- net /esp32/USB_D_N: track 4.05 -> 19.7 mm, vias 0 -> 2
- net /esp32/USB_D_P: track 4.05 -> 19.6 mm, vias 0 -> 2
- net /3v3: track 2.41 -> 10.2 mm, vias 16 -> 13
- net /8v_power/8v_EN: track 0.00 -> 4.47 mm
- net /3v3_power/3v3_SW: track 1.18 -> 5.06 mm
- net /5v_power/5v_SW: track 1.10 -> 4.58 mm
- net /5v_power/5v_out: track 0.30 -> 3.17 mm
- net /VBAT: track 2.71 -> 5.39 mm
- net /esp32/boot0: track 26.6 -> 29.1 mm
- net /STEPPER_MS3: track 154.3 -> 151.9 mm
- net /5v: track 5.99 -> 8.29 mm
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- added copper zone on F.Cu, net /esp32/USB_D_N
- added copper zone on F.Cu, net /esp32/USB_D_P
- added copper zone on In1.Cu, net GND
- removed copper zone on F.Cu, net /motor_driver/REF
- removed copper zone on F.Cu, net /motor_driver1/REF
- removed copper zone on F.Cu, net /motor_driver2/REF
Other:
- board size 105.2 x 89.6 mm -> 103.5 x 89.6 mm
- board text added: "Proto 1"
- board text added: "do-doin' ur mom [sic]"
- board text added: "doin' ur mom"
