File: defcon_badge_main/8v_power.kicad_sch (KiCad schematic)
At the start: 9 parts

Commit message: more layout
Parts:
- C1_V8, C3_V8: footprint PCM_SparkFun-Coil:0805 -> joystick:R_0805_2012Metric_Pad1.20x1.40mm_HandSolder_MINE
- C2_V8: footprint Capacitor_SMD:C_0402_1005Metric -> joystick:R_0402_1005Metric_Pad0.72x0.64mm_HandSolder_MINE
- R1_V8, R2_V8, R3_V8: footprint PCM_SparkFun-Fuse:1206 -> joystick:R_1206_3216Metric_Pad1.30x1.75mm_HandSolder_MINE
Connections:
- net GND: now also U_V8.1 (PGND), U_V8.5 (AGND), U_V8.7 (PAD)
- net 8v_SW: now reaches D_8V1.A, L_V8.2, U_V8.6 (SW)
- net 8v_FB: now reaches C2_V8.1, R2_V8.2, R3_V8.2, U_V8.4 (FB)
- net 8v_EN: now reaches R1_V8.1, U_V8.3 (EN)
Changed lines of the file:
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@@
 		(color 0 0 0 0)
 	)
+	(junction
+		(at 143.51 97.79)
+		(diameter 0)
+		(color 0 0 0 0)
+	)
 	(wire
 		(pts
@@
 	(wire
 		(pts
+			(xy 143.51 97.79) (xy 146.05 97.79)
+		)
+		(stroke
+			(width 0)
+			(type default)
+		)
+	)
+	(wire
+		(pts
 			(xy 116.84 87.63) (xy 116.84 92.71)
 		)
@@
 	(wire
 		(pts
+			(xy 143.51 97.79) (xy 143.51 100.33)
+		)
+		(stroke
+			(width 0)
+			(type default)
+		)
+	)
+	(wire
+		(pts
 			(xy 116.84 87.63) (xy 129.54 87.63)
 		)
@@
 	(wire
 		(pts
+			(xy 140.97 97.79) (xy 143.51 97.79)
+		)
+		(stroke
+			(width 0)
+			(type default)
+		)
+	)
+	(wire
+		(pts
 			(xy 175.26 87.63) (xy 181.61 87.63)
 		)
@@
 			(width 0)
 			(type default)
+		)
+	)
+	(label "8v_VIN"
+		(at 119.38 87.63 0)
+		(effects
+			(font
+				(size 1.27 1.27)
+			)
+			(justify left bottom)
+		)
+	)
+	(label "8v_EN"
+		(at 128.27 92.71 0)
+		(effects
+			(font
+				(size 1.27 1.27)
+			)
+			(justify left bottom)
+		)
+	)
+	(label "8v_FB"
+		(at 154.94 92.71 0)
+		(effects
+			(font
+				(size 1.27 1.27)
+			)
+			(justify left bottom)
+		)
+	)
+	(label "8v_SW"
+		(at 153.67 81.28 0)
+		(effects
+			(font
+				(size 1.27 1.27)
+			)
+			(justify left bottom)
 		)
 	)
@@
 			)
 		)
-		(property "Footprint" "PCM_SparkFun-Fuse:1206"
+		(property "Footprint" "joystick:R_1206_3216Metric_Pad1.30x1.75mm_HandSolder_MINE"
 			(at 157.734 110.236 90)
 			(effects
@@
 			)
 		)
-		(property "Footprint" "PCM_SparkFun-Coil:0805"
+		(property "Footprint" "joystick:R_0805_2012Metric_Pad1.20x1.40mm_HandSolder_MINE"
 			(at 107.6452 95.25 0)
 			(effects
@@
 			)
 		)
-		(property "Footprint" "PCM_SparkFun-Coil:0805"
+		(property "Footprint" "joystick:R_0805_2012Metric_Pad1.20x1.40mm_HandSolder_MINE"
 			(at 176.2252 113.03 0)
 			(effects
@@
 			)
 		)
-		(property "Footprint" "PCM_SparkFun-Fuse:1206"
+		(property "Footprint" "joystick:R_1206_3216Metric_Pad1.30x1.75mm_HandSolder_MINE"
 			(at 168.656 93.726 90)
 			(effects
@@
 			)
 		)
-		(property "Footprint" "Capacitor_SMD:C_0402_1005Metric"
+		(property "Footprint" "joystick:R_0402_1005Metric_Pad0.72x0.64mm_HandSolder_MINE"
 			(at 172.72 101.9048 0)
 			(effects
@@
 			)
 		)
-		(property "Footprint" "PCM_SparkFun-Fuse:1206"
+		(property "Footprint" "joystick:R_1206_3216Metric_Pad1.30x1.75mm_HandSolder_MINE"
 			(at 124.206 93.726 90)
 			(effects
@@
 					(unit 1)
 				)
+			)
+		)
+	)
+	(symbol
+		(lib_id "power:GND")
+		(at 143.51 100.33 0)
+		(unit 1)
+		(exclude_from_sim no)
+		(in_bom yes)
+		(on_board yes)
+		(dnp no)
+		(fields_autoplaced yes)
+		(property "Reference" "#PWR059"
+			(at 143.51 106.68 0)
+			(effects
+				(font
+					(size 1.27 1.27)
+				)
+				(hide yes)
+			)
+		)
+		(property "Value" "GND"
+			(at 143.51 105.41 0)
+			(effects
+				(font
+					(size 1.27 1.27)
+				)
+			)
+		)
+		(property "Footprint" ""
+			(at 143.51 100.33 0)
+			(effects
+				(font
+					(size 1.27 1.27)
+				)
+				(hide yes)
+			)
+		)
+		(property "Datasheet" ""
+			(at 143.51 100.33 0)
+			(effects
+				(font
+					(size 1.27 1.27)
+				)
+				(hide yes)
+			)
+		)
+		(property "Description" "Power symbol creates a global label with name \"GND\" , ground"
+			(at 143.51 100.33 0)
+			(effects
+				(font
+					(size 1.27 1.27)
+				)
+				(hide yes)
+			)
+		)
+		(pin "1"
+		)
+		(instances
+			(project "defcon_badge_main"
+				(path "/b497f1e3-23b9-4176-bc4d-bc3995ba532c/78645551-29a0-445b-ace5-a898bf317411"
+					(reference "#PWR059")
+					(unit 1)
+				)

Commit message: added component parts and modifications
Parts:
- C1_V8, C3_V8: MPN (none) -> GMC21X5R106K16NT; Rating (none) -> 16V
- C2_V8: footprint joystick:R_0402_1005Metric_Pad0.72x0.64mm_HandSolder_MINE -> joystick:R_0603_1608Metric_Pad0.98x0.95mm_HandSolder_MINE; MPN (none) -> GMC10X7R102K16NT
- D_8V1: MPN (none) -> SS24FL
- L_V8: MPN (none) -> 74438357100
- R1_V8: MPN (none) -> RM12F1003CT; TOL (none) -> 1%
- R2_V8: MPN (none) -> RM12F5362CT; TOL (none) -> 1%
- R3_V8: MPN (none) -> RM12F1002CT; TOL (none) -> 1%
- U_V8: MPN (none) -> LMR62421XSD/NOPB
Changed lines of the file:
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@@
 			)
 		)
-		(property "Datasheet" "~"
+		(property "Datasheet" "https://www.we-online.com/components/products/datasheet/74438357100.pdf"
 			(at 139.7 72.39 0)
 			(effects
@@
 					(size 1.27 1.27)
 				)
+			)
+		)
+		(property "MPN" "74438357100 "
+			(at 139.7 72.39 90)
+			(effects
+				(font
+					(size 1.27 1.27)
+				)
+				(hide yes)
 			)
 		)
@@
 			)
 		)
-		(property "Datasheet" "~"
+		(property "Datasheet" "https://calchip.com/wp-content/uploads/2025/05/RMSERIES-052225.pdf"
 			(at 158.75 110.49 0)
 			(effects
@@
 		)
 		(property "Description" "Resistor, US symbol"
+			(at 158.75 110.49 0)
+			(effects
+				(font
+					(size 1.27 1.27)
+				)
+				(hide yes)
+			)
+		)
+		(property "MPN" "RM12F1002CT"
+			(at 158.75 110.49 0)
+			(effects
+				(font
+					(size 1.27 1.27)
+				)
+				(hide yes)
+			)
+		)
+		(property "TOL" "1%"
 			(at 158.75 110.49 0)
 			(effects
@@
 			)
 		)
-		(property "Datasheet" "~"
+		(property "Datasheet" "https://calchip.com/wp-content/uploads/2025/05/GMC-Series-3.pdf"
 			(at 106.68 91.44 0)
 			(effects
@@
 		)
 		(property "Description" "Unpolarized capacitor"
+			(at 106.68 91.44 0)
+			(effects
+				(font
+					(size 1.27 1.27)
+				)
+				(hide yes)
+			)
+		)
+		(property "MPN" "GMC21X5R106K16NT"
+			(at 106.68 91.44 0)
+			(effects
+				(font
+					(size 1.27 1.27)
+				)
+				(hide yes)
+			)
+		)
+		(property "Rating" "16V"
 			(at 106.68 91.44 0)
 			(effects
@@
 			)
 		)
-		(property "Datasheet" "~"
+		(property "Datasheet" "https://calchip.com/wp-content/uploads/2025/05/GMC-Series-3.pdf"
 			(at 175.26 109.22 0)
 			(effects
@@
 		)
 		(property "Description" "Unpolarized capacitor"
+			(at 175.26 109.22 0)
+			(effects
+				(font
+					(size 1.27 1.27)
+				)
+				(hide yes)
+			)
+		)
+		(property "MPN" "GMC21X5R106K16NT"
+			(at 175.26 109.22 0)
+			(effects
+				(font
+					(size 1.27 1.27)
+				)
+				(hide yes)
+			)
+		)
+		(property "Rating" "16V"
 			(at 175.26 109.22 0)
 			(effects
@@
 			)
 		)
-		(property "Datasheet" ""
+		(property "Datasheet" "https://www.onsemi.com/pdf/datasheet/ss26fl-d.pdf"
 			(at 163.83 87.63 0)
 			(effects
@@
 				)
 				(justify bottom)
+				(hide yes)
+			)
+		)
+		(property "MPN" "SS24FL"
+			(at 163.83 87.63 0)
+			(effects
+				(font
+					(size 1.27 1.27)
+				)
 				(hide yes)
 			)
@@
 			)
 		)
+		(property "MPN" "LMR62421XSD/NOPB"
+			(at 143.51 90.17 0)
+			(effects
+				(font
+					(size 1.27 1.27)
+				)
+				(hide yes)
+			)
+		)
 		(pin "5"
 		)
@@
 			)
 		)
-		(property "Datasheet" "~"
+		(property "Datasheet" "https://calchip.com/wp-content/uploads/2025/05/RMSERIES-052225.pdf"
 			(at 168.91 92.71 0)
 			(effects
@@
 		(property "Description" "Resistor, US symbol"
 			(at 168.91 92.71 0)
+			(effects
+				(font
+					(size 1.27 1.27)
+				)
+				(hide yes)
+			)
+		)
+		(property "MPN" "RM12F5362CT"
+			(at 168.91 92.71 90)
+			(effects
+				(font
+					(size 1.27 1.27)
+				)
+				(hide yes)
+			)
+		)
+		(property "TOL" "1%"
+			(at 168.91 92.71 90)
 			(effects
 				(font
@@
 			)
 		)
-		(property "Footprint" "joystick:R_0402_1005Metric_Pad0.72x0.64mm_HandSolder_MINE"
+		(property "Footprint" "joystick:R_0603_1608Metric_Pad0.98x0.95mm_HandSolder_MINE"
 			(at 172.72 101.9048 0)
 			(effects
@@
 			)
 		)
-		(property "Datasheet" "~"
+		(property "Datasheet" "https://calchip.com/wp-content/uploads/2025/05/GMC-Series-3.pdf"
 			(at 168.91 102.87 0)
 			(effects
@@
 		(property "Description" "Unpolarized capacitor"
 			(at 168.91 102.87 0)
+			(effects
+				(font
+					(size 1.27 1.27)
+				)
+				(hide yes)
+			)
+		)
+		(property "MPN" "GMC10X7R102K16NT"
+			(at 168.91 102.87 90)
 			(effects
 				(font
@@
 			)
 		)
-		(property "Datasheet" "~"
+		(property "Datasheet" "https://calchip.com/wp-content/uploads/2025/05/RMSERIES-052225.pdf"
 			(at 124.46 92.71 0)
 			(effects
@@
 			(effects
 				(font
+					(size 1.27 1.27)
+				)
+				(hide yes)
+			)
+		)
+		(property "MPN" "RM12F1003CT"
+			(at 124.46 92.71 90)
+			(effects
+				(font
+					(size 1.27 1.27)
+				)
+				(hide yes)
+			)
+		)
+		(property "TOL" "1%"
+			(at 124.46 92.71 90)
+			(effects
+				(font
