File: defcon_badge_main/led.kicad_sch (KiCad schematic)
At the start: 24 parts, among them J10 Conn_01x02_Pin, J11 Conn_01x02_Pin, J12 Conn_01x02_Pin, J13 Conn_01x02_Pin, J14 Conn_01x02_Pin, J15 Conn_01x02_Pin, J16 Conn_01x02_Pin, J17 Conn_01x02_Pin, J18 Conn_01x02_Pin, J19 Conn_01x02_Pin, J20 Conn_01x02_Pin, J21 Conn_01x02_Pin, J22 Conn_01x02_Pin, J3 Conn_01x02_Pin, J9 Conn_01x02_Pin

Commit message: begin full layout
Parts:
- added J4, J5, J6: Conn_01x02_Pin, Connector_PinHeader_1.00mm:PinHeader_1x02_P1.00mm_Vertical, symbol Connector:Conn_01x02_Pin
Connections:
- net 5v: now also J4.2 (Pin_2), J5.2 (Pin_2), J6.2 (Pin_2)
- net at J10.1 (Pin_1), J11.1 (Pin_1), J12.1 (Pin_1)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: now also J4.1 (Pin_1)
- net at J13.1 (Pin_1), J14.1 (Pin_1), J15.1 (Pin_1)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: now also J5.1 (Pin_1)
- net at J18.1 (Pin_1), J19.1 (Pin_1), J20.1 (Pin_1)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: now also J6.1 (Pin_1)
Other:
- note added: "TODO add more(24)"
- moved on the sheet: J10, J11, J12, J13, J14, J15, J16, J17, J18, J19, J20, J21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

Commit message: more layout
Parts:
- R1_BLED1, R1_GLED1, R1_RLED1, R2_BLED1, R2_GLED1, R2_RLED1: footprint PCM_SparkFun-Fuse:1206 -> joystick:R_1206_3216Metric_Pad1.30x1.75mm_HandSolder_MINE
- renumbered J6 to BLUE_1, J18 to BLUE_2, J19 to BLUE_3, J20 to BLUE_4, J21 to BLUE_5, J22 to BLUE_6, J5 to GREEN_1, J13 to GREEN_2, J14 to GREEN_3, J15 to GREEN_4, J16 to GREEN_5, J17 to GREEN_6, J4 to RED_1, J3 to RED_2, J9 to RED_3, J10 to RED_4, J11 to RED_5, J12 to RED_6
Changed lines of the file:
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@@
 			)
 		)
-		(property "Footprint" "PCM_SparkFun-Fuse:1206"
+		(property "Footprint" "joystick:R_1206_3216Metric_Pad1.30x1.75mm_HandSolder_MINE"
 			(at 64.516 136.144 90)
 			(effects
@@
 		(dnp no)
 		(fields_autoplaced yes)
-		(property "Reference" "J3"
+		(property "Reference" "RED_2"
 			(at 77.47 96.5199 0)
 			(effects
@@
 			(project ""
 				(path "/b497f1e3-23b9-4176-bc4d-bc3995ba532c/6a77c56e-3668-482f-aae0-f4a5bfd6d108"
-					(reference "J3")
+					(reference "RED_2")
 					(unit 1)
 				)
@@
 		(dnp no)
 		(fields_autoplaced yes)
-		(property "Reference" "J9"
+		(property "Reference" "RED_3"
 			(at 77.47 104.1399 0)
 			(effects
@@
 			(project "defcon_badge_main"
 				(path "/b497f1e3-23b9-4176-bc4d-bc3995ba532c/6a77c56e-3668-482f-aae0-f4a5bfd6d108"
-					(reference "J9")
+					(reference "RED_3")
 					(unit 1)
 				)
@@
 		(dnp no)
 		(fields_autoplaced yes)
-		(property "Reference" "J13"
+		(property "Reference" "GREEN_2"
 			(at 160.02 96.5199 0)
 			(effects
@@
 			(project "defcon_badge_main"
 				(path "/b497f1e3-23b9-4176-bc4d-bc3995ba532c/6a77c56e-3668-482f-aae0-f4a5bfd6d108"
-					(reference "J13")
+					(reference "GREEN_2")
 					(unit 1)
 				)
@@
 		(dnp no)
 		(fields_autoplaced yes)
-		(property "Reference" "J17"
+		(property "Reference" "GREEN_6"
 			(at 160.02 126.9999 0)
 			(effects
@@
 			(project "defcon_badge_main"
 				(path "/b497f1e3-23b9-4176-bc4d-bc3995ba532c/6a77c56e-3668-482f-aae0-f4a5bfd6d108"
-					(reference "J17")
+					(reference "GREEN_6")
 					(unit 1)
 				)
@@
 			)
 		)
-		(property "Footprint" "PCM_SparkFun-Fuse:1206"
+		(property "Footprint" "joystick:R_1206_3216Metric_Pad1.30x1.75mm_HandSolder_MINE"
 			(at 147.066 136.144 90)
 			(effects
@@
 		(dnp no)
 		(fields_autoplaced yes)
-		(property "Reference" "J16"
+		(property "Reference" "GREEN_5"
 			(at 160.02 119.3799 0)
 			(effects
@@
 			(project "defcon_badge_main"
 				(path "/b497f1e3-23b9-4176-bc4d-bc3995ba532c/6a77c56e-3668-482f-aae0-f4a5bfd6d108"
-					(reference "J16")
+					(reference "GREEN_5")
 					(unit 1)
 				)
@@
 		(dnp no)
 		(fields_autoplaced yes)
-		(property "Reference" "J20"
+		(property "Reference" "BLUE_4"
 			(at 242.57 111.7599 0)
 			(effects
@@
 			(project "defcon_badge_main"
 				(path "/b497f1e3-23b9-4176-bc4d-bc3995ba532c/6a77c56e-3668-482f-aae0-f4a5bfd6d108"
-					(reference "J20")
+					(reference "BLUE_4")
 					(unit 1)
 				)
@@
 			)
 		)
-		(property "Footprint" "PCM_SparkFun-Fuse:1206"
+		(property "Footprint" "joystick:R_1206_3216Metric_Pad1.30x1.75mm_HandSolder_MINE"
 			(at 204.724 146.304 90)
 			(effects
@@
 		(dnp no)
 		(fields_autoplaced yes)
-		(property "Reference" "J15"
+		(property "Reference" "GREEN_4"
 			(at 160.02 111.7599 0)
 			(effects
@@
 			(project "defcon_badge_main"
 				(path "/b497f1e3-23b9-4176-bc4d-bc3995ba532c/6a77c56e-3668-482f-aae0-f4a5bfd6d108"
-					(reference "J15")
+					(reference "GREEN_4")
 					(unit 1)
 				)
@@
 		(dnp no)
 		(fields_autoplaced yes)
-		(property "Reference" "J11"
+		(property "Reference" "RED_5"
 			(at 77.47 119.3799 0)
 			(effects
@@
 			(project "defcon_badge_main"
 				(path "/b497f1e3-23b9-4176-bc4d-bc3995ba532c/6a77c56e-3668-482f-aae0-f4a5bfd6d108"
-					(reference "J11")
+					(reference "RED_5")
 					(unit 1)
 				)
@@
 		(dnp no)
 		(fields_autoplaced yes)
-		(property "Reference" "J4"
+		(property "Reference" "RED_1"
 			(at 77.47 90.1699 0)
 			(effects
@@
 			(project "defcon_badge_main"
 				(path "/b497f1e3-23b9-4176-bc4d-bc3995ba532c/6a77c56e-3668-482f-aae0-f4a5bfd6d108"
-					(reference "J4")
+					(reference "RED_1")
 					(unit 1)
 				)
@@
 		(dnp no)
 		(fields_autoplaced yes)
-		(property "Reference" "J18"
+		(property "Reference" "BLUE_2"
 			(at 242.57 96.5199 0)
 			(effects
@@
 			(project "defcon_badge_main"
 				(path "/b497f1e3-23b9-4176-bc4d-bc3995ba532c/6a77c56e-3668-482f-aae0-f4a5bfd6d108"
-					(reference "J18")
+					(reference "BLUE_2")
 					(unit 1)
 				)
@@
 		(dnp no)
 		(fields_autoplaced yes)
-		(property "Reference" "J12"
+		(property "Reference" "RED_6"
 			(at 77.47 126.9999 0)
 			(effects
@@
 			(project "defcon_badge_main"
 				(path "/b497f1e3-23b9-4176-bc4d-bc3995ba532c/6a77c56e-3668-482f-aae0-f4a5bfd6d108"
-					(reference "J12")
+					(reference "RED_6")
 					(unit 1)
 				)
@@
 		(dnp no)
 		(fields_autoplaced yes)
-		(property "Reference" "J22"
+		(property "Reference" "BLUE_6"
 			(at 242.57 126.9999 0)
 			(effects
@@
 			(project "defcon_badge_main"
 				(path "/b497f1e3-23b9-4176-bc4d-bc3995ba532c/6a77c56e-3668-482f-aae0-f4a5bfd6d108"
-					(reference "J22")
+					(reference "BLUE_6")
 					(unit 1)
 				)
@@
 		(dnp no)
 		(fields_autoplaced yes)
-		(property "Reference" "J19"
+		(property "Reference" "BLUE_3"
 			(at 242.57 104.1399 0)
 			(effects
@@
 			(project "defcon_badge_main"
 				(path "/b497f1e3-23b9-4176-bc4d-bc3995ba532c/6a77c56e-3668-482f-aae0-f4a5bfd6d108"
-					(reference "J19")
+					(reference "BLUE_3")
 					(unit 1)
 				)
@@
 			)
 		)
-		(property "Footprint" "PCM_SparkFun-Fuse:1206"
+		(property "Footprint" "joystick:R_1206_3216Metric_Pad1.30x1.75mm_HandSolder_MINE"
 			(at 229.616 136.144 90)
 			(effects
@@
 		(dnp no)
 		(fields_autoplaced yes)
-		(property "Reference" "J10"
+		(property "Reference" "RED_4"
 			(at 77.47 111.7599 0)
 			(effects
@@
 			(project "defcon_badge_main"
 				(path "/b497f1e3-23b9-4176-bc4d-bc3995ba532c/6a77c56e-3668-482f-aae0-f4a5bfd6d108"
-					(reference "J10")
+					(reference "RED_4")
 					(unit 1)
 				)
@@
 			)
 		)
-		(property "Footprint" "PCM_SparkFun-Fuse:1206"
+		(property "Footprint" "joystick:R_1206_3216Metric_Pad1.30x1.75mm_HandSolder_MINE"
 			(at 122.174 146.304 90)
 			(effects
@@
 			)
 		)
-		(property "Footprint" "PCM_SparkFun-Fuse:1206"
+		(property "Footprint" "joystick:R_1206_3216Metric_Pad1.30x1.75mm_HandSolder_MINE"
 			(at 44.704 146.304 90)
 			(effects
@@
 		(dnp no)
 		(fields_autoplaced yes)
-		(property "Reference" "J6"
+		(property "Reference" "BLUE_1"
 			(at 242.57 90.1699 0)
 			(effects
@@
 			(project "defcon_badge_main"
 				(path "/b497f1e3-23b9-4176-bc4d-bc3995ba532c/6a77c56e-3668-482f-aae0-f4a5bfd6d108"
-					(reference "J6")
+					(reference "BLUE_1")
 					(unit 1)
 				)
@@
 		(dnp no)
 		(fields_autoplaced yes)
-		(property "Reference" "J5"
+		(property "Reference" "GREEN_1"
 			(at 160.02 90.1699 0)
 			(effects
@@
 			(project "defcon_badge_main"
 				(path "/b497f1e3-23b9-4176-bc4d-bc3995ba532c/6a77c56e-3668-482f-aae0-f4a5bfd6d108"
-					(reference "J5")
+					(reference "GREEN_1")
 					(unit 1)
 				)
@@
 		(dnp no)
 		(fields_autoplaced yes)
-		(property "Reference" "J21"
+		(property "Reference" "BLUE_5"
 			(at 242.57 119.3799 0)
 			(effects
@@
 			(project "defcon_badge_main"
 				(path "/b497f1e3-23b9-4176-bc4d-bc3995ba532c/6a77c56e-3668-482f-aae0-f4a5bfd6d108"
-					(reference "J21")
+					(reference "BLUE_5")
 					(unit 1)
 				)
@@
 		(dnp no)
 		(fields_autoplaced yes)
-		(property "Reference" "J14"
+		(property "Reference" "GREEN_3"
 			(at 160.02 104.1399 0)
 			(effects
@@
 			(project "defcon_badge_main"
 				(path "/b497f1e3-23b9-4176-bc4d-bc3995ba532c/6a77c56e-3668-482f-aae0-f4a5bfd6d108"
-					(reference "J14")
-					(unit 1)
-				)
+					(reference "GREEN_3")
+					(unit 1)
+				)

Commit message: moar layout
Parts:
- R1_BLED1, R1_GLED1, R1_RLED1, R2_BLED1, R2_GLED1, R2_RLED1: footprint joystick:R_1206_3216Metric_Pad1.30x1.75mm_HandSolder_MINE -> joystick:R_0805_2012Metric_Pad1.20x1.40mm_HandSolder
Connections:
- net LED_R_POW: now reaches Q_RLED1.1 (C), R2_RLED1.2
- net LED_G_POW: now reaches Q_GLED1.1 (C), R2_GLED1.2
- net LED_B_SIG: now reaches Q_BLED1.2 (B), R1_BLED1.2
- net LED_R_SIG: now reaches Q_RLED1.2 (B), R1_RLED1.2
- net LED_B_POW: now reaches Q_BLED1.1 (C), R2_BLED1.2
- net LED_G_SIG: now reaches Q_GLED1.2 (B), R1_GLED1.2
Changed lines of the file:
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@@
+		)
+	)
+	(label "LED_B_POW"
+		(at 228.6 142.24 0)
+		(effects
+			(font
+				(size 1.27 1.27)
+			)
+			(justify left bottom)
+		)
+	)
+	(label "LED_B_SIG"
+		(at 209.55 147.32 0)
+		(effects
+			(font
+				(size 1.27 1.27)
+			)
+			(justify left bottom)
+		)
+	)
+	(label "LED_G_SIG"
+		(at 127 147.32 0)
+		(effects
+			(font
+				(size 1.27 1.27)
+			)
+			(justify left bottom)
+		)
+	)
+	(label "LED_R_POW"
+		(at 63.5 140.97 0)
+		(effects
+			(font
+				(size 1.27 1.27)
+			)
+			(justify left bottom)
+		)
+	)
+	(label "LED_R_SIG"
+		(at 49.53 147.32 0)
+		(effects
+			(font
+				(size 1.27 1.27)
+			)
+			(justify left bottom)
+		)
+	)
+	(label "LED_G_POW"
+		(at 146.05 142.24 0)
+		(effects
+			(font
+				(size 1.27 1.27)
+			)
+			(justify left bottom)
 		)
 	)
@@
 			)
 		)
-		(property "Footprint" "joystick:R_1206_3216Metric_Pad1.30x1.75mm_HandSolder_MINE"
+		(property "Footprint" "joystick:R_0805_2012Metric_Pad1.20x1.40mm_HandSolder"
 			(at 64.516 136.144 90)
 			(effects
@@
 			)
 		)
-		(property "Footprint" "joystick:R_1206_3216Metric_Pad1.30x1.75mm_HandSolder_MINE"
+		(property "Footprint" "joystick:R_0805_2012Metric_Pad1.20x1.40mm_HandSolder"
 			(at 147.066 136.144 90)
 			(effects
@@
 			)
 		)
-		(property "Footprint" "joystick:R_1206_3216Metric_Pad1.30x1.75mm_HandSolder_MINE"
+		(property "Footprint" "joystick:R_0805_2012Metric_Pad1.20x1.40mm_HandSolder"
 			(at 204.724 146.304 90)
 			(effects
@@
 			)
 		)
-		(property "Footprint" "joystick:R_1206_3216Metric_Pad1.30x1.75mm_HandSolder_MINE"
+		(property "Footprint" "joystick:R_0805_2012Metric_Pad1.20x1.40mm_HandSolder"
 			(at 229.616 136.144 90)
 			(effects
@@
 			)
 		)
-		(property "Footprint" "joystick:R_1206_3216Metric_Pad1.30x1.75mm_HandSolder_MINE"
+		(property "Footprint" "joystick:R_0805_2012Metric_Pad1.20x1.40mm_HandSolder"
 			(at 122.174 146.304 90)
 			(effects
@@
 			)
 		)
-		(property "Footprint" "joystick:R_1206_3216Metric_Pad1.30x1.75mm_HandSolder_MINE"
+		(property "Footprint" "joystick:R_0805_2012Metric_Pad1.20x1.40mm_HandSolder"
 			(at 44.704 146.304 90)
 			(effects

Commit message: added component parts and modifications
Parts:
- BLUE_1, BLUE_2, BLUE_3, BLUE_4, BLUE_5, BLUE_6, GREEN_1, GREEN_2, GREEN_3, GREEN_4, GREEN_5, GREEN_6, RED_1, RED_2, RED_3, RED_4, RED_5, RED_6: now not fitted
- Q_BLED1, Q_GLED1, Q_RLED1: footprint joystick:npn -> joystick:SOT-23-3; MPN (none) -> MMUN2211LT1G
- R1_BLED1, R1_GLED1, R1_RLED1: MPN (none) -> RM10F1501CT; TOL (none) -> 1%
- R2_BLED1, R2_GLED1, R2_RLED1: MPN (none) -> RM10F2200CT; TOL (none) -> 1%
Changed lines of the file:
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@@
 			)
 		)
-		(property "Datasheet" "~"
+		(property "Datasheet" "https://calchip.com/wp-content/uploads/2025/05/RMSERIES-052225.pdf"
 			(at 63.5 135.89 0)
 			(effects
@@
 			)
 		)
+		(property "MPN" "RM10F2200CT"
+			(at 63.5 135.89 0)
+			(effects
+				(font
+					(size 1.27 1.27)
+				)
+				(hide yes)
+			)
+		)
+		(property "TOL" "1%"
+			(at 63.5 135.89 0)
+			(effects
+				(font
+					(size 1.27 1.27)
+				)
+				(hide yes)
+			)
+		)
 		(pin "1"
 		)
@@
 		(in_bom yes)
 		(on_board yes)
-		(dnp no)
+		(dnp yes)
 		(fields_autoplaced yes)
 		(property "Reference" "RED_2"
@@
 		(in_bom yes)
 		(on_board yes)
-		(dnp no)
+		(dnp yes)
 		(fields_autoplaced yes)
 		(property "Reference" "RED_3"
@@
 		(in_bom yes)
 		(on_board yes)
-		(dnp no)
+		(dnp yes)
 		(fields_autoplaced yes)
 		(property "Reference" "GREEN_2"
@@
 		(in_bom yes)
 		(on_board yes)
-		(dnp no)
+		(dnp yes)
 		(fields_autoplaced yes)
 		(property "Reference" "GREEN_6"
@@
 			)
 		)
-		(property "Datasheet" "~"
+		(property "Datasheet" "https://calchip.com/wp-content/uploads/2025/05/RMSERIES-052225.pdf"
 			(at 146.05 135.89 0)
 			(effects
@@
 			)
 		)
+		(property "MPN" "RM10F2200CT"
+			(at 146.05 135.89 0)
+			(effects
+				(font
+					(size 1.27 1.27)
+				)
+				(hide yes)
+			)
+		)
+		(property "TOL" "1%"
+			(at 146.05 135.89 0)
+			(effects
+				(font
+					(size 1.27 1.27)
+				)
+				(hide yes)
+			)
+		)
 		(pin "1"
 		)
@@
 		(in_bom yes)
 		(on_board yes)
-		(dnp no)
+		(dnp yes)
 		(fields_autoplaced yes)
 		(property "Reference" "GREEN_5"
@@
 		(in_bom yes)
 		(on_board yes)
-		(dnp no)
+		(dnp yes)
 		(fields_autoplaced yes)
 		(property "Reference" "BLUE_4"
@@
 			)
 		)
-		(property "Datasheet" "~"
+		(property "Datasheet" "https://calchip.com/wp-content/uploads/2025/05/RMSERIES-052225.pdf"
 			(at 204.47 147.32 0)
 			(effects
@@
 			)
 		)
+		(property "MPN" "RM10F1501CT"
+			(at 204.47 147.32 90)
+			(effects
+				(font
+					(size 1.27 1.27)
+				)
+				(hide yes)
+			)
+		)
+		(property "TOL" "1%"
+			(at 204.47 147.32 90)
+			(effects
+				(font
+					(size 1.27 1.27)
+				)
+				(hide yes)
+			)
+		)
 		(pin "2"
 		)
@@
 			)
 		)
-		(property "Footprint" "joystick:npn"
+		(property "Footprint" "joystick:SOT-23-3"
 			(at 124.46 147.32 0)
 			(effects
@@
 			)
 		)
+		(property "MPN" "MMUN2211LT1G"
+			(at 60.96 147.32 0)
+			(effects
+				(font
+					(size 1.27 1.27)
+				)
+				(hide yes)
+			)
+		)
 		(pin "1"
 		)
@@
 		(in_bom yes)
 		(on_board yes)
-		(dnp no)
+		(dnp yes)
 		(fields_autoplaced yes)
 		(property "Reference" "GREEN_4"
@@
 		(in_bom yes)
 		(on_board yes)
-		(dnp no)
+		(dnp yes)
 		(fields_autoplaced yes)
 		(property "Reference" "RED_5"
@@
 		(in_bom yes)
 		(on_board yes)
-		(dnp no)
+		(dnp yes)
 		(fields_autoplaced yes)
 		(property "Reference" "RED_1"
@@
 		(in_bom yes)
 		(on_board yes)
-		(dnp no)
+		(dnp yes)
 		(fields_autoplaced yes)
 		(property "Reference" "BLUE_2"
@@
 		(in_bom yes)
 		(on_board yes)
-		(dnp no)
+		(dnp yes)
 		(fields_autoplaced yes)
 		(property "Reference" "RED_6"
@@
 		(in_bom yes)
 		(on_board yes)
-		(dnp no)
+		(dnp yes)
 		(fields_autoplaced yes)
 		(property "Reference" "BLUE_6"
@@
 		(in_bom yes)
 		(on_board yes)
-		(dnp no)
+		(dnp yes)
 		(fields_autoplaced yes)
 		(property "Reference" "BLUE_3"
@@
 			)
 		)
-		(property "Datasheet" "~"
+		(property "Datasheet" "https://calchip.com/wp-content/uploads/2025/05/RMSERIES-052225.pdf"
 			(at 228.6 135.89 0)
 			(effects
@@
 			)
 		)
+		(property "MPN" "RM10F2200CT"
+			(at 228.6 135.89 0)
+			(effects
+				(font
+					(size 1.27 1.27)
+				)
+				(hide yes)
+			)
+		)
+		(property "TOL" "1%"
+			(at 228.6 135.89 0)
+			(effects
+				(font
+					(size 1.27 1.27)
+				)
+				(hide yes)
+			)
+		)
 		(pin "1"
 		)
@@
 		(in_bom yes)
 		(on_board yes)
-		(dnp no)
+		(dnp yes)
 		(fields_autoplaced yes)
 		(property "Reference" "RED_4"
@@
 			)
 		)
-		(property "Datasheet" "~"
+		(property "Datasheet" "https://calchip.com/wp-content/uploads/2025/05/RMSERIES-052225.pdf"
 			(at 121.92 147.32 0)
 			(effects
@@
 			)
 		)
+		(property "MPN" "RM10F1501CT"
+			(at 121.92 147.32 90)
+			(effects
+				(font
+					(size 1.27 1.27)
+				)
+				(hide yes)
+			)
+		)
+		(property "TOL" "1%"
+			(at 121.92 147.32 90)
+			(effects
+				(font
+					(size 1.27 1.27)
+				)
+				(hide yes)
+			)
+		)
 		(pin "2"
 		)
@@
 			)
 		)
-		(property "Footprint" "joystick:npn"
+		(property "Footprint" "joystick:SOT-23-3"
 			(at 207.01 147.32 0)
 			(effects
@@
 			)
 		)
+		(property "MPN" "MMUN2211LT1G"
+			(at 143.51 147.32 0)
+			(effects
+				(font
+					(size 1.27 1.27)
+				)
+				(hide yes)
+			)
+		)
 		(pin "1"
 		)
@@
 			)
 		)
-		(property "Datasheet" "~"
+		(property "Datasheet" "https://calchip.com/wp-content/uploads/2025/05/RMSERIES-052225.pdf"
 			(at 44.45 147.32 0)
 			(effects
@@
 			)
 		)
+		(property "MPN" "RM10F1501CT"
+			(at 44.45 147.32 90)
+			(effects
+				(font
+					(size 1.27 1.27)
+				)
+				(hide yes)
+			)
+		)
+		(property "TOL" "1%"
+			(at 44.45 147.32 90)
+			(effects
+				(font
+					(size 1.27 1.27)
+				)
+				(hide yes)
+			)
+		)
 		(pin "2"
 		)
@@
 		(in_bom yes)
 		(on_board yes)
-		(dnp no)
+		(dnp yes)
 		(fields_autoplaced yes)
 		(property "Reference" "BLUE_1"
@@
 		(in_bom yes)
 		(on_board yes)
-		(dnp no)
+		(dnp yes)
 		(fields_autoplaced yes)
 		(property "Reference" "GREEN_1"
@@
 		(in_bom yes)
 		(on_board yes)
-		(dnp no)
+		(dnp yes)
 		(fields_autoplaced yes)
 		(property "Reference" "BLUE_5"
@@
 		(in_bom yes)
 		(on_board yes)
-		(dnp no)
+		(dnp yes)
 		(fields_autoplaced yes)
 		(property "Reference" "GREEN_3"
@@
 			)
 		)
-		(property "Footprint" "joystick:npn"
+		(property "Footprint" "joystick:SOT-23-3"
 			(at 289.56 147.32 0)
 			(effects
@@
 			(at 226.06 147.32 0)
 			(effects
+				(font
+					(size 1.27 1.27)
+				)
+				(hide yes)
+			)
+		)
+		(property "MPN" "MMUN2211LT1G"
+			(at 226.06 147.32 0)
+			(effects
