File: defcon_badge_main/power_regulator.kicad_sch (KiCad schematic)
At the start: 6 parts

Commit message: more layout
Parts:
- C1_V3, C2_V3: footprint PCM_SparkFun-Coil:0805 -> joystick:R_0805_2012Metric_Pad1.20x1.40mm_HandSolder_MINE
- R1_V3, R2_V3: footprint PCM_SparkFun-Fuse:1206 -> joystick:R_1206_3216Metric_Pad1.30x1.75mm_HandSolder_MINE
Connections:
- net 3v3_FB: now reaches R1_V3.2, R2_V3.1, U_3V1.1 (FB)
- net 3v3_SW: now reaches L_V3.2, U_3V1.5 (SW)
Changed lines of the file:
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@@
+		)
+	)
+	(label "3v3_FB"
+		(at 156.21 109.22 0)
+		(effects
+			(font
+				(size 1.27 1.27)
+			)
+			(justify left bottom)
+		)
+	)
+	(label "3v3_SW"
+		(at 153.67 59.69 0)
+		(effects
+			(font
+				(size 1.27 1.27)
+			)
+			(justify left bottom)
 		)
 	)
@@
 			)
 		)
-		(property "Footprint" "PCM_SparkFun-Coil:0805"
+		(property "Footprint" "joystick:R_0805_2012Metric_Pad1.20x1.40mm_HandSolder_MINE"
 			(at 88.5952 101.6 0)
 			(effects
@@
 			)
 		)
-		(property "Footprint" "PCM_SparkFun-Fuse:1206"
+		(property "Footprint" "joystick:R_1206_3216Metric_Pad1.30x1.75mm_HandSolder_MINE"
 			(at 168.656 101.854 90)
 			(effects
@@
 			)
 		)
-		(property "Footprint" "PCM_SparkFun-Fuse:1206"
+		(property "Footprint" "joystick:R_1206_3216Metric_Pad1.30x1.75mm_HandSolder_MINE"
 			(at 168.656 117.094 90)
 			(effects
@@
 			)
 		)
-		(property "Footprint" "PCM_SparkFun-Coil:0805"
+		(property "Footprint" "joystick:R_0805_2012Metric_Pad1.20x1.40mm_HandSolder_MINE"
 			(at 185.1152 113.03 0)
 			(effects

Commit message: added component parts and modifications
Parts:
- C1_V3: MPN (none) -> GMC21X5R106K16NT; Rating (none) -> 16V
- C2_V3: MPN (none) -> GMC10Y5V475Z6R3NT; Rating (none) -> 16V
- L_V3: MPN (none) -> 74479288147
- R1_V3: MPN (none) -> RM12F4533CT; TOL (none) -> 1%
- R2_V3: MPN (none) -> RM12F1003CT; TOL (none) -> 1%
- U_3V1: MPN (none) -> TPS61023DRLR
Changed lines of the file:
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@@
 			)
 		)
-		(property "Datasheet" "~"
+		(property "Datasheet" "https://calchip.com/wp-content/uploads/2025/05/GMC-Series-3.pdf"
 			(at 87.63 97.79 0)
 			(effects
@@
 		)
 		(property "Description" "Unpolarized capacitor"
+			(at 87.63 97.79 0)
+			(effects
+				(font
+					(size 1.27 1.27)
+				)
+				(hide yes)
+			)
+		)
+		(property "MPN" "GMC21X5R106K16NT"
+			(at 87.63 97.79 0)
+			(effects
+				(font
+					(size 1.27 1.27)
+				)
+				(hide yes)
+			)
+		)
+		(property "Rating" "16V"
 			(at 87.63 97.79 0)
 			(effects
@@
 			)
 		)
-		(property "Datasheet" "~"
+		(property "Datasheet" "https://calchip.com/wp-content/uploads/2025/05/RMSERIES-052225.pdf"
 			(at 167.64 101.6 0)
 			(effects
@@
 		)
 		(property "Description" "Resistor, US symbol"
+			(at 167.64 101.6 0)
+			(effects
+				(font
+					(size 1.27 1.27)
+				)
+				(hide yes)
+			)
+		)
+		(property "MPN" "RM12F4533CT"
+			(at 167.64 101.6 0)
+			(effects
+				(font
+					(size 1.27 1.27)
+				)
+				(hide yes)
+			)
+		)
+		(property "TOL" "1%"
 			(at 167.64 101.6 0)
 			(effects
@@
 			)
 		)
-		(property "Datasheet" "~"
+		(property "Datasheet" "https://calchip.com/wp-content/uploads/2025/05/RMSERIES-052225.pdf"
 			(at 167.64 116.84 0)
 			(effects
@@
 		)
 		(property "Description" "Resistor, US symbol"
+			(at 167.64 116.84 0)
+			(effects
+				(font
+					(size 1.27 1.27)
+				)
+				(hide yes)
+			)
+		)
+		(property "MPN" "RM12F1003CT"
+			(at 167.64 116.84 0)
+			(effects
+				(font
+					(size 1.27 1.27)
+				)
+				(hide yes)
+			)
+		)
+		(property "TOL" "1%"
 			(at 167.64 116.84 0)
 			(effects
@@
 			)
 		)
-		(property "Datasheet" "~"
+		(property "Datasheet" "https://calchip.com/wp-content/uploads/2025/05/GMC-Series-3.pdf"
 			(at 184.15 109.22 0)
 			(effects
@@
 		)
 		(property "Description" "Unpolarized capacitor"
+			(at 184.15 109.22 0)
+			(effects
+				(font
+					(size 1.27 1.27)
+				)
+				(hide yes)
+			)
+		)
+		(property "MPN" "GMC10Y5V475Z6R3NT"
+			(at 184.15 109.22 0)
+			(effects
+				(font
+					(size 1.27 1.27)
+				)
+				(hide yes)
+			)
+		)
+		(property "Rating" "16V"
 			(at 184.15 109.22 0)
 			(effects
@@
 			)
 		)
-		(property "Datasheet" "~"
+		(property "Datasheet" "https://www.we-online.com/components/products/datasheet/74479288147.pdf"
 			(at 130.81 59.69 0)
 			(effects
@@
 					(size 1.27 1.27)
 				)
+			)
+		)
+		(property "MPN" "74479288147"
+			(at 130.81 59.69 90)
+			(effects
+				(font
+					(size 1.27 1.27)
+				)
+				(hide yes)
 			)
 		)
@@
 			)
 		)
-		(property "Datasheet" ""
+		(property "Datasheet" "https://www.ti.com/lit/ds/symlink/tps61023.pdf?HQS=dis-dk-null-digikeymode-dsf-pf-null-wwe&ts=1777151769302&ref_url=https%253A%252F%252Fwww.ti.com%252Fgeneral%252Fdocs%252Fsuppproductinfo.tsp%253FdistId%253D10%2526gotoUrl%253Dhttps%253A%252F%252Fwww.ti.com%252Flit%252Fgpn%252Ftps61023"
 			(at 132.08 96.52 0)
 			(effects
@@
 				(hide yes)
 			)
+		)
+		(property "MPN" "TPS61023DRLR"
+			(at 132.08 96.52 0)
+			(effects
+				(font
+					(size 1.27 1.27)
+				)
+				(hide yes)
+			)
